File: _autosave-lamp.kicad_sch (KiCad schematic)
At the start: 18 parts, among them J1 Screw_Terminal_01x02, J2 Screw_Terminal_01x02, Q1 2N7002, U1 ESP-12E, U2 34.81-7048, U3 AMS1117-3.3

Commit message: some chnges
some changes
Connections:
- net at J1.1 (Pin_1), PS1.2 (AC/N), RV1.1: now also J2.2 (Pin_2); no longer J2.1 (Pin_1)
- net at F1.1: now also J2.1 (Pin_1); no longer J2.2 (Pin_2)
Other:
- moved on the sheet: J2
Changed lines of the file:
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@@
+    (stroke (width 0) (type default) (color 0 0 0 0))
+  )
+  (wire (pts (xy 58.42 101.6) (xy 63.5 101.6))
     (stroke (width 0) (type default) (color 0 0 0 0))
   )
@@
   )
   (wire (pts (xy 171.45 137.16) (xy 171.45 138.43))
-    (stroke (width 0) (type default) (color 0 0 0 0))
-  )
-  (wire (pts (xy 58.42 101.6) (xy 63.5 101.6))
     (stroke (width 0) (type default) (color 0 0 0 0))
   )
@@
     (pin "2")
   )
-  (symbol (lib_id "Connector:Screw_Terminal_01x02") (at 53.34 101.6 0) (mirror y) (unit 1)
+  (symbol (lib_id "Connector:Screw_Terminal_01x02") (at 53.34 104.14 180) (unit 1)
     (in_bom yes) (on_board yes) (fields_autoplaced)
     (property "Reference" "J2" (id 0) (at 53.34 95.25 0))
     (property "Value" "Screw_Terminal_01x02" (id 1) (at 53.34 97.79 0))
-    (property "Footprint" "TerminalBlock:TerminalBlock_Altech_AK300-2_P5.00mm" (id 2) (at 53.34 101.6 0)
-      (effects (font (size 1.27 1.27)) hide)
-    )
-    (property "Datasheet" "~" (id 3) (at 53.34 101.6 0)
-      (effects (font (size 1.27 1.27)) hide)
-    )
+    (property "Footprint" "TerminalBlock:TerminalBlock_Altech_AK300-2_P5.00mm" (id 2) (at 53.34 104.14 0)
+      (effects (font (size 1.27 1.27)) hide)
+    )
+    (property "Datasheet" "~" (id 3) (at 53.34 104.14 0)
+      (effects (font (size 1.27 1.27)) hide)
+    )
